File: cpu_board.kicad_pcb (KiCad board)
At the start: 10 copper layers, 80 x 100 mm, 501 parts, among them J1 JXK0-0190NL, J10 EJ508A, J11 DNP-PH1RB-05-UA, J12 TBP03R1-350-02BE, J14 2PH1R-05-UA, J16 0791091011, J17 TBP03R1-350-02BE, J2 BMODE, J20 USB4105-GF-A, J3 JTAG, J4 USB4105-GF-A, J5 2PH1-02-UA, J6 DNP-PH1RB-09-UA, J7 TSW-102-07-F-S, J8 2PH2R-10-UA, J9 SM04B-SRSS-TB, K1 1462042-3, Q1 PSMN075-100MSE, Q10 FJV992FMTF, Q11 XP10TN135N, Q12 BSZ520N15NS3G, Q13 MMBT3906, Q14 FDMC86160, Q15 MMBT3904, Q16 PUMH13, Q2 PSMN075-100MSE, Q3 PSMN075-100MSE, Q4 PSMN075-100MSE, Q5 PSMN075-100MSE, Q6 PSMN075-100MSE, Q7 PSMN075-100MSE, Q8 PSMN075-100MSE, Q9 PSMN075-100MSE, T1 750310742, T2 PE-68386NL, U1 LT4321IUF_PBF, U10 ADP5054ACPZ-R7, U11 SP3003-02JTG, U12 MIC2025-2YMM-TR, U13 SN74LVC2G241DCUR, U15 MAX31875R0TZS_T, U16 MX52LM04A11XSI, U17 W25Q128JVPIM, U2 ADSP-SC573KBCZ-3, U3 SI5351B-B-GM, U32 ADIN1300CCPZ, U33 ADP123AUJZ-R7, U34 ESDA5V3SC6, U36 SP3003-02JTG, U38 CP2102N-A02-GQFN24R, U4 ADM6315, U5 MIC5166YML-TR, U6 IS43TR16128DL-125KBL, U7 LT4276BIUFDTRPBF, U8 ESDA5V3SC6, U9 MOC207M, Y1 25 Mhz, Y2 25 Mhz, Y3 25 Mhz

Commit message: post prototype build edits clean U32 under ic edits beef up relay traces
Parts:
- R71: value 53.2K -> 52.3K
- moved C249 0.46 mm to (208.9, 90.0), turned to 0 degrees
- moved C255 0.33 mm to (211.5, 86.5)
- moved C240 0.28 mm to (209.4, 92.9)
- moved C242 0.28 mm to (210.5, 93.0)
- moved C238 0.28 mm to (213.1, 93.0)
- moved C236 0.25 mm to (211.8, 93.5)
- moved C235 0.25 mm to (214.5, 94.7)
- moved C245 0.25 mm to (214.2, 93.0)
- moved R241 0.20 mm to (217.4, 88.1)
- moved C250 0.20 mm to (217.4, 88.1)
- moved C254 0.10 mm to (217.4, 89.2)
- moved R240 0.10 mm to (217.4, 89.2)
- turned C248 to 0 degrees
Routing:
- net GND: track 351.3 -> 362.2 mm, vias 277 -> 283
- net Net-(Q16B-COLLECTOR): track 27.7 -> 23.4 mm
- net /Ethernet/PHY_CFG1: track 14.0 -> 16.9 mm
- net ETH0_MDC: track 49.6 -> 50.9 mm
- net /Ethernet/GIGe_LINK: track 5.69 -> 4.51 mm
- net +3V3: track 208.4 -> 209.1 mm
- net Net-(C53-Pad1): track 25.7 -> 25.0 mm
- net RELAY_DRV: track 86.7 -> 86.2 mm
- net +0v9: track 16.0 -> 16.5 mm, vias 7 -> 6
