File: poe_controller.kicad_sch (KiCad schematic)
At the start: 78 parts, among them Q10 FJV992FMTF, Q11 XP10TN135N, Q12 BSZ520N15NS3G, Q13 MMBT3906, Q14 FDMC86160, Q15 MMBT3904, Q9 PSMN075-100MSE, T1 750310742, T2 PE-68386NL, U7 LT4276BIUFDTRPBF, U9 MOC207M

Commit message: post prototype build edits clean U32 under ic edits beef up relay traces
Parts:
- R71: value 53.2K -> 52.3K; Manufacturer KOA -> TE Connectivity Passive Product; Part Number RN73H1JTTD5232F100 -> CPF0603F52K3C1
- R73: Manufacturer KOA -> Vishay; Part Number RN73H1JTTD3301F100 -> MCT06030C3301FP500
- R84: Manufacturer KOA -> Yageo; Part Number RN73H1JTTD2612F100 -> RT0603BRD0726K1L
Changed lines of the file:
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@@
 			)
 		)
-		(property "Manufacturer" "KOA"
+		(property "Manufacturer" "Vishay"
 			(at 88.9 50.8 0)
 			(hide yes)
@@
 			)
 		)
-		(property "Part Number" "RN73H1JTTD3301F100"
+		(property "Part Number" "MCT06030C3301FP500"
 			(at 88.9 50.8 0)
 			(hide yes)
@@
 			)
 		)
-		(property "Manufacturer" "KOA"
+		(property "Manufacturer" "Yageo"
 			(at 195.58 133.35 0)
 			(hide yes)
@@
 			)
 		)
-		(property "Part Number" "RN73H1JTTD2612F100"
+		(property "Part Number" "RT0603BRD0726K1L"
 			(at 195.58 133.35 0)
 			(hide yes)
@@
 			)
 		)
-		(property "Value" "53.2K"
+		(property "Value" "52.3K"
 			(at 63.754 99.06 0)
 			(show_name no)
@@
 			)
 		)
-		(property "Manufacturer" "KOA"
+		(property "Manufacturer" "TE Connectivity Passive Product"
 			(at 64.77 101.6 0)
 			(hide yes)
@@
 			)
 		)
-		(property "Part Number" "RN73H1JTTD5232F100"
+		(property "Part Number" "CPF0603F52K3C1"
 			(at 64.77 101.6 0)
 			(hide yes)
