File: io_connectors.kicad_sch (KiCad schematic)
At the start: 39 parts, among them J10 EJ508A, J11 DNP-PH1RB-05-UA, J12 TBP03R1-350-02BE, J14 2PH1R-05-UA, J16 0791091011, J17 TBP03R1-350-02BE, J5 2PH1-02-UA, J6 DNP-PH1RB-09-UA, J7 TSW-102-07-F-S, J8 2PH2R-10-UA, J9 SM04B-SRSS-TB, K1 1462042-3, Q16 PUMH13, U13 SN74LVC2G241DCUR, U15 MAX31875R0TZS_T

Commit message: fix range and relay connector part numbers
Parts:
- J14: value 2PH1R-05-UA -> 2PH1-05-UA; Part Number 2PH1R-05-UA -> 2PH1-05-UA
- J8: value 2PH2R-10-UA -> 2PH2-10-UA; Part Number 2PH2R-10-UA -> 2PH2-10-UA
Changed lines of the file:
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@@
 			)
 		)
-		(property "Value" "2PH2R-10-UA"
+		(property "Value" "2PH2-10-UA"
 			(at 55.88 120.65 0)
 			(show_name no)
@@
 			)
 		)
-		(property "Datasheet" "https://app.adam-tech.com/products/download/data_sheet/199986/2ph2r-xx-ua-data-sheet.pdf"
+		(property "Datasheet" "https://app.adam-tech.com/products/download/data_sheet/200454/2ph2-xx-ua-data-sheet.pdf"
 			(at 54.61 129.54 0)
 			(hide yes)
@@
 			)
 		)
-		(property "Part Number" "2PH2R-10-UA"
+		(property "Part Number" "2PH2-10-UA"
 			(at 54.61 129.54 0)
 			(hide yes)
@@
 			)
 		)
-		(property "Value" "2PH1R-05-UA"
+		(property "Value" "2PH1-05-UA"
 			(at 153.67 132.0801 0)
 			(show_name no)
@@
 			)
 		)
-		(property "Datasheet" "https://www.adafruit.com/product/6250"
+		(property "Datasheet" "https://app.adam-tech.com/products/download/data_sheet/200457/2ph1-xx-ua-data-sheet.pdf"
 			(at 151.13 134.62 0)
 			(hide yes)
@@
 			)
 		)
-		(property "Part Number" "2PH1R-05-UA"
+		(property "Part Number" "2PH1-05-UA"
 			(at 151.13 134.62 0)
 			(hide yes)
